File: PCB/KeyBoard.kicad_pcb (KiCad board)
At the start: 2 copper layers, 346.1 x 96.6 mm, 205 parts, among them P1 USB_C_Plug_USB2.0, P2 USB_C_Plug_USB2.0, SW1 SW_Push, SW10 SW_Push, SW11 SW_Push, SW12 SW_Push, SW13 SW_Push, SW14 SW_Push, SW15 SW_Push, SW16 SW_Push, SW17 SW_Push, SW18 SW_Push, SW19 SW_Push, SW2 SW_Push, SW20 SW_Push, SW21 SW_Push, SW22 SW_Push, SW23 SW_Push, SW24 SW_Push, SW25 SW_Push, SW26 SW_Push, SW27 SW_Push, SW28 SW_Push, SW29 SW_Push, SW3 SW_Push, SW30 SW_Push, SW31 SW_Push, SW32 SW_Push, SW33 SW_Push, SW34 SW_Push, SW35 SW_Push, SW36 SW_Push, SW37 SW_Push, SW38 SW_Push, SW39 SW_Push, SW4 SW_Push, SW40 SW_Push, SW41 SW_Push, SW42 SW_Push, SW43 SW_Push, SW44 SW_Push, SW45 SW_Push, SW46 SW_Push, SW47 SW_Push, SW48 SW_Push, SW49 SW_Push, SW5 SW_Push, SW50 SW_Push, SW51 SW_Push, SW52 SW_Push, SW53 SW_Push, SW54 SW_Push, SW55 SW_Push, SW56 SW_Push, SW57 SW_Push, SW58 SW_Push, SW59 SW_Push, SW6 SW_Push, SW60 SW_Push, SW61 SW_Push, SW64 RotaryEncoder_Switch_MP, SW7 SW_Push, SW8 SW_Push, SW9 SW_Push, U1 PCA9555D, U2 PCA9555D, U3 XIAO-RP2040-DIP

Commit message: Add files via upload
Parts:
- D100, D101, D102, D103, D104, D105, D106, D107, D108, D109, D110, D111, D112, D113, D114, D115, D116, D117, D118, D119, D120, D121, D122, D123, D63, D64, D65, D66, D67, D68, D69, D70, D71, D72, D73, D74, D75, D76, D77, D78, D79, D80, D81, D82, D83, D84, D85, D86, D87, D88, D89, D90, D91, D92, D93, D94, D95, D96, D97, D98, D99: footprint SK6812-E (2):LED_SK6812-E -> Sk6812-MINI-E:LED-SMD_4P-L3.2-W2.8-LS5.9_SK6812MINI-E; moved to B.Cu
- moved D103 16.3 mm to (298.1, 111.9), turned to 180 degrees
- moved D16 16.3 mm to (88.6, 115.5)
- moved D22 16.3 mm to (262.8, 115.8)
- moved D45 16.3 mm to (148.1, 172.5)
- moved D2 16.3 mm to (77.3, 96.3)
- moved D3 16.3 mm to (98.2, 96.5)
- moved D30 16.3 mm to (95.0, 134.4)
- moved D52 16.3 mm to (123.0, 153.5)
- moved D64 16.3 mm to (75.5, 92.7), turned to 180 degrees
- moved D67 16.3 mm to (133.1, 92.5), turned to 180 degrees
- moved D92 16.3 mm to (83.1, 168.7), turned to 180 degrees
- moved REF** 16.3 mm to (95.0, 163.6)
- moved SW17 16.3 mm to (106.9, 102.1)
- moved SW32 16.3 mm to (130.7, 121.2)
- moved SW50 16.3 mm to (71.2, 140.2)
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Routing:
- net +5V: track 50.3 -> 255.8 mm, vias 38 -> 37
- net +5LV: track 31.6 -> 164.4 mm
- net +3.3V: track 179.2 -> 279.3 mm, vias 14 -> 2
- net GNDL: track 176.5 -> 88.7 mm, vias 20 -> 40
- net Net-(D90-DOUT): track 187.2 -> 152.8 mm, vias 2 -> 8
- net GND: track 267.3 -> 235.4 mm, vias 31 -> 52
- net C2: track 143.1 -> 114.5 mm, vias 13 -> 1
- net R1: track 192.0 -> 163.8 mm, vias 6 -> 4
- net Net-(D118-DOUT): track 136.2 -> 163.4 mm, vias 8 -> 4
- net LEDR: track 145.1 -> 118.6 mm, vias 2 -> 5
- net C8: track 147.0 -> 124.5 mm, vias 11 -> 0
- net Net-(D100-DOUT): track 122.6 -> 102.5 mm, vias 4 -> 2
- net SCRLin: track 207.4 -> 225.5 mm, vias 2 -> 0
- net Net-(D107-DOUT): track 150.2 -> 132.4 mm, vias 4 -> 2
- net C10: track 177.1 -> 159.6 mm, vias 15 -> 4
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
Commit message: Add files via upload
Parts:
- removed D100, D101, D102, D103, D104, D105, D106, D107, D108, D109, D110, D111, D112, D113, D114, D115, D116, D117, D118, D119, D120, D121, D122, D123, D63, D64, D65, D66, D67, D68, D69, D70, D71, D72, D73, D74, D75, D76, D77, D78, D79, D80, D81, D82, D83, D84, D85, D86, D87, D88, D89, D90, D91, D92, D93, D94, D95, D96, D97, D98, D99: SK6812MINI, Sk6812-MINI-E:LED-SMD_4P-L3.2-W2.8-LS5.9_SK6812MINI-E
- added LED1: SK6812MINI-E_C5149201, Sk6812-MINI-E:LED-SMD_4P-L3.2-W2.8-LS5.9_SK6812MINI-E, B.Cu at (56.9, 92.5)
- added LED10: SK6812MINI-E_C5149201, Sk6812-MINI-E:LED-SMD_4P-L3.2-W2.8-LS5.9_SK6812MINI-E, B.Cu at (104.5, 111.7)
- added LED11: SK6812MINI-E_C5149201, Sk6812-MINI-E:LED-SMD_4P-L3.2-W2.8-LS5.9_SK6812MINI-E, B.Cu at (123.5, 111.5)
- added LED12: SK6812MINI-E_C5149201, Sk6812-MINI-E:LED-SMD_4P-L3.2-W2.8-LS5.9_SK6812MINI-E, B.Cu at (142.5, 111.5)
- added LED13: SK6812MINI-E_C5149201, Sk6812-MINI-E:LED-SMD_4P-L3.2-W2.8-LS5.9_SK6812MINI-E, B.Cu at (161.6, 111.6)
- added LED14: SK6812MINI-E_C5149201, Sk6812-MINI-E:LED-SMD_4P-L3.2-W2.8-LS5.9_SK6812MINI-E, B.Cu at (180.7, 111.7)
- added LED15: SK6812MINI-E_C5149201, Sk6812-MINI-E:LED-SMD_4P-L3.2-W2.8-LS5.9_SK6812MINI-E, B.Cu at (63.9, 130.6)
- added LED16: SK6812MINI-E_C5149201, Sk6812-MINI-E:LED-SMD_4P-L3.2-W2.8-LS5.9_SK6812MINI-E, B.Cu at (90.0, 130.5)
- added LED17: SK6812MINI-E_C5149201, Sk6812-MINI-E:LED-SMD_4P-L3.2-W2.8-LS5.9_SK6812MINI-E, B.Cu at (109.2, 130.6)
- added LED18: SK6812MINI-E_C5149201, Sk6812-MINI-E:LED-SMD_4P-L3.2-W2.8-LS5.9_SK6812MINI-E, B.Cu at (128.3, 130.6)
- added LED19: SK6812MINI-E_C5149201, Sk6812-MINI-E:LED-SMD_4P-L3.2-W2.8-LS5.9_SK6812MINI-E, B.Cu at (147.4, 130.6)
- added LED2: SK6812MINI-E_C5149201, Sk6812-MINI-E:LED-SMD_4P-L3.2-W2.8-LS5.9_SK6812MINI-E, B.Cu at (76.2, 92.5)
- added LED20: SK6812MINI-E_C5149201, Sk6812-MINI-E:LED-SMD_4P-L3.2-W2.8-LS5.9_SK6812MINI-E, B.Cu at (166.3, 130.7)
- added LED21: SK6812MINI-E_C5149201, Sk6812-MINI-E:LED-SMD_4P-L3.2-W2.8-LS5.9_SK6812MINI-E, B.Cu at (185.3, 130.6)
- added LED22: SK6812MINI-E_C5149201, Sk6812-MINI-E:LED-SMD_4P-L3.2-W2.8-LS5.9_SK6812MINI-E, B.Cu at (68.7, 149.7)
- added LED23: SK6812MINI-E_C5149201, Sk6812-MINI-E:LED-SMD_4P-L3.2-W2.8-LS5.9_SK6812MINI-E, B.Cu at (99.6, 149.7)
- added LED24: SK6812MINI-E_C5149201, Sk6812-MINI-E:LED-SMD_4P-L3.2-W2.8-LS5.9_SK6812MINI-E, B.Cu at (118.8, 149.6)
- added LED25: SK6812MINI-E_C5149201, Sk6812-MINI-E:LED-SMD_4P-L3.2-W2.8-LS5.9_SK6812MINI-E, B.Cu at (137.7, 149.7)
- added LED26: SK6812MINI-E_C5149201, Sk6812-MINI-E:LED-SMD_4P-L3.2-W2.8-LS5.9_SK6812MINI-E, B.Cu at (156.7, 149.6)
- added LED27: SK6812MINI-E_C5149201, Sk6812-MINI-E:LED-SMD_4P-L3.2-W2.8-LS5.9_SK6812MINI-E, B.Cu at (175.7, 149.9)
- added LED28: SK6812MINI-E_C5149201, Sk6812-MINI-E:LED-SMD_4P-L3.2-W2.8-LS5.9_SK6812MINI-E, B.Cu at (194.8, 149.5)
- added LED29: SK6812MINI-E_C5149201, Sk6812-MINI-E:LED-SMD_4P-L3.2-W2.8-LS5.9_SK6812MINI-E, B.Cu at (59.2, 168.6)
- added LED3: SK6812MINI-E_C5149201, Sk6812-MINI-E:LED-SMD_4P-L3.2-W2.8-LS5.9_SK6812MINI-E, B.Cu at (94.8, 92.5)
- added LED30: SK6812MINI-E_C5149201, Sk6812-MINI-E:LED-SMD_4P-L3.2-W2.8-LS5.9_SK6812MINI-E, B.Cu at (83.2, 168.7)
- added LED31: SK6812MINI-E_C5149201, Sk6812-MINI-E:LED-SMD_4P-L3.2-W2.8-LS5.9_SK6812MINI-E, B.Cu at (107.0, 168.9)
- added LED32: SK6812MINI-E_C5149201, Sk6812-MINI-E:LED-SMD_4P-L3.2-W2.8-LS5.9_SK6812MINI-E, B.Cu at (145.2, 168.8)
- added LED33: SK6812MINI-E_C5149201, Sk6812-MINI-E:LED-SMD_4P-L3.2-W2.8-LS5.9_SK6812MINI-E, B.Cu at (249.5, 92.9)
- added LED34: SK6812MINI-E_C5149201, Sk6812-MINI-E:LED-SMD_4P-L3.2-W2.8-LS5.9_SK6812MINI-E, B.Cu at (269.1, 92.7)
- added LED35: SK6812MINI-E_C5149201, Sk6812-MINI-E:LED-SMD_4P-L3.2-W2.8-LS5.9_SK6812MINI-E, B.Cu at (287.6, 92.7)
- added LED36: SK6812MINI-E_C5149201, Sk6812-MINI-E:LED-SMD_4P-L3.2-W2.8-LS5.9_SK6812MINI-E, B.Cu at (307.1, 92.8)
- added LED37: SK6812MINI-E_C5149201, Sk6812-MINI-E:LED-SMD_4P-L3.2-W2.8-LS5.9_SK6812MINI-E, B.Cu at (326.0, 92.8)
- added LED38: SK6812MINI-E_C5149201, Sk6812-MINI-E:LED-SMD_4P-L3.2-W2.8-LS5.9_SK6812MINI-E, B.Cu at (345.0, 92.8)
- added LED39: SK6812MINI-E_C5149201, Sk6812-MINI-E:LED-SMD_4P-L3.2-W2.8-LS5.9_SK6812MINI-E, B.Cu at (260.1, 111.7)
- added LED4: SK6812MINI-E_C5149201, Sk6812-MINI-E:LED-SMD_4P-L3.2-W2.8-LS5.9_SK6812MINI-E, B.Cu at (113.8, 92.5)
- added LED40: SK6812MINI-E_C5149201, Sk6812-MINI-E:LED-SMD_4P-L3.2-W2.8-LS5.9_SK6812MINI-E, B.Cu at (278.5, 111.9)
- added LED41: SK6812MINI-E_C5149201, Sk6812-MINI-E:LED-SMD_4P-L3.2-W2.8-LS5.9_SK6812MINI-E, B.Cu at (297.4, 111.8)
- added LED42: SK6812MINI-E_C5149201, Sk6812-MINI-E:LED-SMD_4P-L3.2-W2.8-LS5.9_SK6812MINI-E, B.Cu at (316.7, 111.9)
- added LED43: SK6812MINI-E_C5149201, Sk6812-MINI-E:LED-SMD_4P-L3.2-W2.8-LS5.9_SK6812MINI-E, B.Cu at (335.7, 111.9)
- added LED44: SK6812MINI-E_C5149201, Sk6812-MINI-E:LED-SMD_4P-L3.2-W2.8-LS5.9_SK6812MINI-E, B.Cu at (354.6, 111.9)
- added LED45: SK6812MINI-E_C5149201, Sk6812-MINI-E:LED-SMD_4P-L3.2-W2.8-LS5.9_SK6812MINI-E, B.Cu at (378.9, 111.8)
- added LED46: SK6812MINI-E_C5149201, Sk6812-MINI-E:LED-SMD_4P-L3.2-W2.8-LS5.9_SK6812MINI-E, B.Cu at (264.1, 130.6)
- added LED47: SK6812MINI-E_C5149201, Sk6812-MINI-E:LED-SMD_4P-L3.2-W2.8-LS5.9_SK6812MINI-E, B.Cu at (283.3, 131.2)
- added LED48: SK6812MINI-E_C5149201, Sk6812-MINI-E:LED-SMD_4P-L3.2-W2.8-LS5.9_SK6812MINI-E, B.Cu at (301.9, 130.8)
- added LED49: SK6812MINI-E_C5149201, Sk6812-MINI-E:LED-SMD_4P-L3.2-W2.8-LS5.9_SK6812MINI-E, B.Cu at (321.6, 130.8)
- added LED5: SK6812MINI-E_C5149201, Sk6812-MINI-E:LED-SMD_4P-L3.2-W2.8-LS5.9_SK6812MINI-E, B.Cu at (132.9, 92.5)
- added LED50: SK6812MINI-E_C5149201, Sk6812-MINI-E:LED-SMD_4P-L3.2-W2.8-LS5.9_SK6812MINI-E, B.Cu at (340.2, 130.8)
- added LED51: SK6812MINI-E_C5149201, Sk6812-MINI-E:LED-SMD_4P-L3.2-W2.8-LS5.9_SK6812MINI-E, B.Cu at (371.5, 130.8)
- added LED52: SK6812MINI-E_C5149201, Sk6812-MINI-E:LED-SMD_4P-L3.2-W2.8-LS5.9_SK6812MINI-E, B.Cu at (273.9, 150.1)
- added LED53: SK6812MINI-E_C5149201, Sk6812-MINI-E:LED-SMD_4P-L3.2-W2.8-LS5.9_SK6812MINI-E, B.Cu at (292.5, 149.9)
- added LED54: SK6812MINI-E_C5149201, Sk6812-MINI-E:LED-SMD_4P-L3.2-W2.8-LS5.9_SK6812MINI-E, B.Cu at (311.7, 150.0)
- added LED55: SK6812MINI-E_C5149201, Sk6812-MINI-E:LED-SMD_4P-L3.2-W2.8-LS5.9_SK6812MINI-E, B.Cu at (331.2, 150.0)
- added LED57: SK6812MINI-E_C5149201, Sk6812-MINI-E:LED-SMD_4P-L3.2-W2.8-LS5.9_SK6812MINI-E, B.Cu at (366.7, 149.9)
- added LED58: SK6812MINI-E_C5149201, Sk6812-MINI-E:LED-SMD_4P-L3.2-W2.8-LS5.9_SK6812MINI-E, B.Cu at (271.8, 168.9)
- added LED59: SK6812MINI-E_C5149201, Sk6812-MINI-E:LED-SMD_4P-L3.2-W2.8-LS5.9_SK6812MINI-E, B.Cu at (309.4, 169.0)
- added LED6: SK6812MINI-E_C5149201, Sk6812-MINI-E:LED-SMD_4P-L3.2-W2.8-LS5.9_SK6812MINI-E, B.Cu at (151.9, 92.5)
- added LED61: SK6812MINI-E_C5149201, Sk6812-MINI-E:LED-SMD_4P-L3.2-W2.8-LS5.9_SK6812MINI-E, B.Cu at (333.4, 168.9)
- added LED62: SK6812MINI-E_C5149201, Sk6812-MINI-E:LED-SMD_4P-L3.2-W2.8-LS5.9_SK6812MINI-E, B.Cu at (357.0, 169.0)
- added LED63: SK6812MINI-E_C5149201, Sk6812-MINI-E:LED-SMD_4P-L3.2-W2.8-LS5.9_SK6812MINI-E, B.Cu at (381.1, 168.8)
- added LED7: SK6812MINI-E_C5149201, Sk6812-MINI-E:LED-SMD_4P-L3.2-W2.8-LS5.9_SK6812MINI-E, B.Cu at (171.1, 92.5)
- added LED8: SK6812MINI-E_C5149201, Sk6812-MINI-E:LED-SMD_4P-L3.2-W2.8-LS5.9_SK6812MINI-E, B.Cu at (61.2, 111.6)
- added LED9: SK6812MINI-E_C5149201, Sk6812-MINI-E:LED-SMD_4P-L3.2-W2.8-LS5.9_SK6812MINI-E, B.Cu at (85.2, 111.5)
Routing:
- net +5V: track 255.8 -> 60.9 mm, vias 37 -> 41
- net GND: track 235.4 -> 66.1 mm, vias 52 -> 22
- net Net-(D118-DOUT): track 163.4 -> 0.00 mm, vias 4 -> 0
- net Net-(LED28-DOUT): track 0.00 -> 159.2 mm, vias 0 -> 10
- net Net-(D90-DOUT): track 152.8 -> 0.00 mm, vias 8 -> 0
- net Net-(D69-DOUT): track 150.4 -> 0.00 mm, vias 4 -> 0
- net Net-(D76-DOUT): track 141.5 -> 0.00 mm, vias 4 -> 0
- net Net-(D83-DOUT): track 137.9 -> 0.00 mm, vias 4 -> 0
- net Net-(D107-DOUT): track 132.4 -> 0.00 mm, vias 2 -> 0
- net +5LV: track 164.4 -> 33.0 mm, vias 36 -> 38
- net Net-(LED45-DOUT): track 0.00 -> 128.9 mm, vias 0 -> 4
- net Net-(LED14-DOUT): track 0.00 -> 124.3 mm, vias 0 -> 8
- net Net-(LED21-DOUT): track 0.00 -> 120.1 mm, vias 0 -> 4
- net Net-(D113-DOUT): track 119.9 -> 0.00 mm, vias 8 -> 0
- net Net-(LED7-DOUT): track 0.00 -> 114.2 mm, vias 0 -> 4
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- added copper zone on F.Cu, net +5LV
- added copper zone on F.Cu, net +5V
- added copper zone on B.Cu, net GND
- added copper zone on B.Cu, net GNDL
- removed copper zone on B.Cu, net +5LV
- removed copper zone on B.Cu, net +5V
- removed copper zone on F.Cu, net GND
- removed copper zone on F.Cu, net GNDL
